File: Pinecone_Logger_kicad_project/Logger_KicadProject.sch (KiCad schematic (older format))
At the start: 48 parts, among them J1 PJ-102A, J2 M50-3600542, J3 OSTVN06A150, J4 OSTVN06A150, J5 OSTVN06A150, J6 OSTVN06A150, J7 DM3AT-SF-PEJM5, J8 10_Pin_Header, Q1 AO3420, Q2 AO3420, U1 SAMD20E18A-A, U2 DS3231, U3 AP2281, U4 MIC5211, U5 MAX31856, U6 MAX4618

Commit message: reorganized schematic, getting ready for publication
Parts:
- C11, C12, C13, C14, C15, C16, C17, C2, C4, C5, C7, C8: Capacitance .1uF -> 0.1uF
- C18, C19: Capacitance .01uF -> 0.01uF
- R10: Resistance 68 Ohm -> 120Ω
Connections:
- net +3V3: now also R1.2; no longer R1.1
- net GND: no longer C10.1, C9.1
- net RESET: now also R1.1; no longer R1.2
- net at R10.2: now also U1.1 (XIN32/TC2WO0/SERCOM1P0/PA00); no longer D1.2 (A)
- net STATUS_LED: no longer names the net of R10.1
- net STATUS_LED: now also D1.2 (A); no longer U1.1 (XIN32/TC2WO0/SERCOM1P0/PA00)
- new net: C10.1, C9.1
Other:
- note added: "3v3 and 5v switching.\nUses two AP2281 load switches. \nPlace close to regulator, to shut \noff power to larger areas of board.\n"
- note added: "MCU and related external components."
- note added: "Ports for Dendrometers.\nData pins connected \nto analog inputs."
- note added: "Real Time Clock"
- note added: "Thermocouple System. Multiplexes 4 \ndifferential TCs into an amplifier."
- note removed: "3v3 and 5v switching.\nUses two AP2281 load switches. \nPlace close to regulator, to shut off power to larger areas of board.\n"
- note removed: "Ports for Dendrometers.\nData pins connected to analog inputs."
- note removed: "RTC, other only IC with unswitched power"
- moved on the sheet: BT1, C1, C10, C11, C12, C13, C14, C15, C16, C17, C18, C19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
